Commit message: update moveit config

File: sawyer_moveit_config/srdf/rethink_electric_gripper.srdf.xacro (robot description, xacro)
@@ -6,48 +6,61 @@
 <robot xmlns:xacro="http://www.ros.org/wiki/xacro" name="rethink_electric_gripper">
     <xacro:macro name="rethink_electric_gripper" params="side">
-    <disable_collisions link1="${side}_l6" link2="${side}_gripper_base" reason="Adjacent" />
-    <disable_collisions link1="${side}_gripper_base" link2="${side}_gripper_tip" reason="Adjacent" />
-    <disable_collisions link1="${side}_gripper_tip" link2="${side}_hand" reason="Adjacent" />
-    <disable_collisions link1="${side}_hand" link2="${side}_gripper_base" reason="Adjacent" />
-    <disable_collisions link1="${side}_hand" link2="${side}_connector_plate_base" reason="Adjacent" />
-    <disable_collisions link1="${side}_hand" link2="${side}_electric_gripper_base" reason="Adjacent" />
-    <disable_collisions link1="${side}_gripper_base" link2="${side}_gripper_l_finger" reason="Adjacent" />
-    <disable_collisions link1="${side}_gripper_base" link2="${side}_gripper_l_finger_tip" reason="Never" />
-    <disable_collisions link1="${side}_gripper_base" link2="${side}_gripper_r_finger" reason="Adjacent" />
-    <disable_collisions link1="${side}_gripper_base" link2="${side}_gripper_r_finger_tip" reason="Never" />
-    <disable_collisions link1="${side}_gripper_base" link2="${side}_connector_plate_base" reason="Adjacent" />
-    <disable_collisions link1="${side}_gripper_base" link2="${side}_electric_gripper_base" reason="Adjacent" />
-    <disable_collisions link1="${side}_connector_plate_base" link2="${side}_gripper_l_finger" reason="Adjacent" />
-    <disable_collisions link1="${side}_connector_plate_base" link2="${side}_gripper_l_finger_tip" reason="Never" />
-    <disable_collisions link1="${side}_connector_plate_base" link2="${side}_gripper_r_finger" reason="Adjacent" />
-    <disable_collisions link1="${side}_connector_plate_base" link2="${side}_gripper_r_finger_tip" reason="Never" />
-    <disable_collisions link1="${side}_electric_gripper_base" link2="${side}_connector_plate_base" reason="Adjacent" />
-    <disable_collisions link1="${side}_electric_gripper_base" link2="${side}_gripper_l_finger" reason="Adjacent" />
-    <disable_collisions link1="${side}_electric_gripper_base" link2="${side}_gripper_l_finger_tip" reason="Never" />
-    <disable_collisions link1="${side}_electric_gripper_base" link2="${side}_gripper_r_finger" reason="Adjacent" />
-    <disable_collisions link1="${side}_electric_gripper_base" link2="${side}_gripper_r_finger_tip" reason="Never" />
-    <disable_collisions link1="${side}_gripper_tip" link2="${side}_gripper_l_finger" reason="Default" />
-    <disable_collisions link1="${side}_gripper_tip" link2="${side}_gripper_l_finger_tip" reason="Never" />
-    <disable_collisions link1="${side}_gripper_tip" link2="${side}_gripper_r_finger" reason="Default" />
-    <disable_collisions link1="${side}_gripper_tip" link2="${side}_gripper_r_finger_tip" reason="Never" />
-    <disable_collisions link1="${side}_gripper_l_finger" link2="${side}_gripper_l_finger_tip" reason="Adjacent" />
-    <disable_collisions link1="${side}_gripper_l_finger" link2="${side}_gripper_r_finger" reason="Never" />
-    <disable_collisions link1="${side}_gripper_l_finger" link2="${side}_gripper_r_finger_tip" reason="Never" />
-    <disable_collisions link1="${side}_gripper_l_finger" link2="${side}_hand" reason="Never" />
-    <disable_collisions link1="${side}_gripper_l_finger" link2="${side}_hand_camera" reason="Never" />
-    <disable_collisions link1="${side}_gripper_l_finger_tip" link2="${side}_gripper_r_finger" reason="Never" />
-    <disable_collisions link1="${side}_gripper_l_finger_tip" link2="${side}_hand" reason="Never" />
-    <disable_collisions link1="${side}_gripper_l_finger_tip" link2="${side}_hand_camera" reason="Never" />
-    <disable_collisions link1="${side}_gripper_l_finger_tip" link2="${side}_wrist" reason="Never" />
-    <disable_collisions link1="${side}_gripper_r_finger" link2="${side}_gripper_r_finger_tip" reason="Adjacent" />
-    <disable_collisions link1="${side}_gripper_r_finger" link2="${side}_hand" reason="Never" />
-    <disable_collisions link1="${side}_gripper_r_finger" link2="${side}_hand_camera" reason="Never" />
-    <disable_collisions link1="${side}_gripper_r_finger" link2="${side}_wrist" reason="Never" />
-    <disable_collisions link1="${side}_gripper_r_finger_tip" link2="${side}_hand" reason="Never" />
-    <disable_collisions link1="${side}_gripper_r_finger_tip" link2="${side}_hand_camera" reason="Never" />
-    <disable_collisions link1="${side}_gripper_r_finger_tip" link2="${side}_wrist" reason="Never" />
-    <disable_collisions link1="${side}_gripper_l_finger_tip" link2="${side}_gripper_r_finger_tip" reason="Never" />
-    <disable_collisions link1="${side}_gripper_l_finger" link2="${side}_gripper_l_finger_tip" reason="Never" />
-    <disable_collisions link1="${side}_gripper_r_finger" link2="${side}_gripper_r_finger_tip" reason="Never" />
+        <group name="hand">
+            <joint name="${side}_gripper_l_finger_joint"/>
+            <joint name="${side}_gripper_r_finger_joint"/>
+            <!-- <joint name="right_hand"/> -->
+        </group>
+        <group_state name="open" group="hand">
+            <joint name="${side}_gripper_l_finger_joint" value="0.0416" />
+            <!-- <joint name="right_gripper_r_finger_joint" value="0.0416" /> -->
+        </group_state>
+        <group_state name="close" group="hand">
+            <joint name="${side}_gripper_l_finger_joint" value="0.0" />
+            <!-- <joint name="right_gripper_r_finger_joint" value="0.0" /> -->
+        </group_state>
+        <disable_collisions link1="${side}_l6" link2="${side}_gripper_base" reason="Adjacent" />
+        <disable_collisions link1="${side}_gripper_base" link2="${side}_gripper_tip" reason="Adjacent" />
+        <disable_collisions link1="${side}_gripper_tip" link2="${side}_hand" reason="Adjacent" />
+        <disable_collisions link1="${side}_hand" link2="${side}_gripper_base" reason="Adjacent" />
+        <disable_collisions link1="${side}_hand" link2="${side}_connector_plate_base" reason="Adjacent" />
+        <disable_collisions link1="${side}_hand" link2="${side}_electric_gripper_base" reason="Adjacent" />
+        <disable_collisions link1="${side}_gripper_base" link2="${side}_gripper_l_finger" reason="Adjacent" />
+        <disable_collisions link1="${side}_gripper_base" link2="${side}_gripper_l_finger_tip" reason="Never" />
+        <disable_collisions link1="${side}_gripper_base" link2="${side}_gripper_r_finger" reason="Adjacent" />
+        <disable_collisions link1="${side}_gripper_base" link2="${side}_gripper_r_finger_tip" reason="Never" />
+        <disable_collisions link1="${side}_gripper_base" link2="${side}_connector_plate_base" reason="Adjacent" />
+        <disable_collisions link1="${side}_gripper_base" link2="${side}_electric_gripper_base" reason="Adjacent" />
+        <disable_collisions link1="${side}_connector_plate_base" link2="${side}_gripper_l_finger" reason="Adjacent" />
+        <disable_collisions link1="${side}_connector_plate_base" link2="${side}_gripper_l_finger_tip" reason="Never" />
+        <disable_collisions link1="${side}_connector_plate_base" link2="${side}_gripper_r_finger" reason="Adjacent" />
+        <disable_collisions link1="${side}_connector_plate_base" link2="${side}_gripper_r_finger_tip" reason="Never" />
+        <disable_collisions link1="${side}_electric_gripper_base" link2="${side}_connector_plate_base" reason="Adjacent" />
+        <disable_collisions link1="${side}_electric_gripper_base" link2="${side}_gripper_l_finger" reason="Adjacent" />
+        <disable_collisions link1="${side}_electric_gripper_base" link2="${side}_gripper_l_finger_tip" reason="Never" />
+        <disable_collisions link1="${side}_electric_gripper_base" link2="${side}_gripper_r_finger" reason="Adjacent" />
+        <disable_collisions link1="${side}_electric_gripper_base" link2="${side}_gripper_r_finger_tip" reason="Never" />
+        <disable_collisions link1="${side}_gripper_tip" link2="${side}_gripper_l_finger" reason="Default" />
+        <disable_collisions link1="${side}_gripper_tip" link2="${side}_gripper_l_finger_tip" reason="Never" />
+        <disable_collisions link1="${side}_gripper_tip" link2="${side}_gripper_r_finger" reason="Default" />
+        <disable_collisions link1="${side}_gripper_tip" link2="${side}_gripper_r_finger_tip" reason="Never" />
+        <disable_collisions link1="${side}_gripper_l_finger" link2="${side}_gripper_l_finger_tip" reason="Adjacent" />
+        <disable_collisions link1="${side}_gripper_l_finger" link2="${side}_gripper_r_finger" reason="Never" />
+        <disable_collisions link1="${side}_gripper_l_finger" link2="${side}_gripper_r_finger_tip" reason="Never" />
+        <disable_collisions link1="${side}_gripper_l_finger" link2="${side}_hand" reason="Never" />
+        <disable_collisions link1="${side}_gripper_l_finger" link2="${side}_hand_camera" reason="Never" />
+        <disable_collisions link1="${side}_gripper_l_finger_tip" link2="${side}_gripper_r_finger" reason="Never" />
+        <disable_collisions link1="${side}_gripper_l_finger_tip" link2="${side}_hand" reason="Never" />
+        <disable_collisions link1="${side}_gripper_l_finger_tip" link2="${side}_hand_camera" reason="Never" />
+        <disable_collisions link1="${side}_gripper_l_finger_tip" link2="${side}_wrist" reason="Never" />
+        <disable_collisions link1="${side}_gripper_r_finger" link2="${side}_gripper_r_finger_tip" reason="Adjacent" />
+        <disable_collisions link1="${side}_gripper_r_finger" link2="${side}_hand" reason="Never" />
+        <disable_collisions link1="${side}_gripper_r_finger" link2="${side}_hand_camera" reason="Never" />
+        <disable_collisions link1="${side}_gripper_r_finger" link2="${side}_wrist" reason="Never" />
+        <disable_collisions link1="${side}_gripper_r_finger_tip" link2="${side}_hand" reason="Never" />
+        <disable_collisions link1="${side}_gripper_r_finger_tip" link2="${side}_hand_camera" reason="Never" />
+        <disable_collisions link1="${side}_gripper_r_finger_tip" link2="${side}_wrist" reason="Never" />
+        <disable_collisions link1="${side}_gripper_l_finger_tip" link2="${side}_gripper_r_finger_tip" reason="Never" />
+        <disable_collisions link1="${side}_gripper_l_finger" link2="${side}_gripper_l_finger_tip" reason="Never" />
+        <disable_collisions link1="${side}_gripper_r_finger" link2="${side}_gripper_r_finger_tip" reason="Never" />
     </xacro:macro>
 </robot>

File: sawyer_moveit_config/srdf/sawyer_base.srdf.xacro (robot description, xacro)
@@ -22,16 +22,25 @@
     group names-->
     <group name="right_arm">
-        <chain base_link="base" tip_link="$(arg tip_name)" />
+      <chain base_link="base" tip_link="$(arg tip_name)" />
     </group>
     <!--GROUP STATES: Purpose: Define a named state for a particular group, in
     terms of joint values. This is useful to define states like 'folded arms'-->
     <group_state name="zero_pose" group="right_arm">
-        <joint name="right_j0" value="0" />
-        <joint name="right_j1" value="0" />
-        <joint name="right_j2" value="0" />
-        <joint name="right_j3" value="0" />
-        <joint name="right_j4" value="0" />
-        <joint name="right_j5" value="0" />
-        <joint name="right_j6" value="0" />
+      <joint name="right_j0" value="0" />
+      <joint name="right_j1" value="0" />
+      <joint name="right_j2" value="0" />
+      <joint name="right_j3" value="0" />
+      <joint name="right_j4" value="0" />
+      <joint name="right_j5" value="0" />
+      <joint name="right_j6" value="0" />
+    </group_state>
+    <group_state name="ready" group="right_arm">
+      <joint name="right_j0" value="0.136716796875"/>
+      <joint name="right_j1" value="-1.345919921875"/>
+      <joint name="right_j2" value="-0.3328642578125"/>
+      <joint name="right_j3" value="2.0867880859375"/>
+      <joint name="right_j4" value="-0.19401171875"/>
+      <joint name="right_j5" value="-0.8204111328125"/>
+      <joint name="right_j6" value="-1.0447021484375"/>
     </group_state>
     <!--VIRTUAL JOINT: Purpose: this element defines a virtual joint between a
